File: Jitter_Cleaner.kicad_sch (KiCad schematic)
At the start: 44 parts, among them T1 TCM2-43X+, T3 TCM2-43X+, U18 SI5394, U20 TLV75733PDBV, U21 TLV75718PDBV, Y1 CX3225SB48000D0FPJC1

Commit message: Changes to Power Filtering
- Removed extra bulk caps on FMC power inputs
- Cleaned up some power routing between U22 & U44
- Made some vias larger for power tree connections
- Changed 22uF to a new 35V part
- Changed 10uF part to a new equivalent part due to OOS.
- Modified text near U27 on schematic for clarity
- Added notes on the power schematics showing effective capacitance of chosen bulk mlcc caps
Parts:
- C143, C46, C47, C50, C51, C63, C73: MPN GRM21BR61E106KA73L -> TMK212BBJ106MG-T; Manufacturer Murata -> Taiyo Yuden
Changed lines of the file:
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@@
 			)
 		)
-		(property "MPN" "GRM21BR61E106KA73L"
+		(property "MPN" "TMK212BBJ106MG-T"
 			(at 194.31 54.61 0)
 			(effects
@@
 			)
 		)
-		(property "Manufacturer" "Murata"
+		(property "Manufacturer" "Taiyo Yuden"
 			(at 194.31 54.61 0)
 			(effects
@@
 			)
 		)
-		(property "MPN" "GRM21BR61E106KA73L"
+		(property "MPN" "TMK212BBJ106MG-T"
 			(at 298.45 54.61 0)
 			(effects
@@
 			)
 		)
-		(property "Manufacturer" "Murata"
+		(property "Manufacturer" "Taiyo Yuden"
 			(at 298.45 54.61 0)
 			(effects
@@
 			)
 		)
-		(property "MPN" "GRM21BR61E106KA73L"
+		(property "MPN" "TMK212BBJ106MG-T"
 			(at 248.92 55.88 0)
 			(effects
@@
 			)
 		)
-		(property "Manufacturer" "Murata"
+		(property "Manufacturer" "Taiyo Yuden"
 			(at 248.92 55.88 0)
 			(effects
@@
 			)
 		)
-		(property "MPN" "GRM21BR61E106KA73L"
+		(property "MPN" "TMK212BBJ106MG-T"
 			(at 175.26 88.9 0)
 			(effects
@@
 			)
 		)
-		(property "Manufacturer" "Murata"
+		(property "Manufacturer" "Taiyo Yuden"
 			(at 175.26 88.9 0)
 			(effects
@@
 			)
 		)
-		(property "MPN" "GRM21BR61E106KA73L"
+		(property "MPN" "TMK212BBJ106MG-T"
 			(at 143.51 55.88 0)
 			(effects
@@
 			)
 		)
-		(property "Manufacturer" "Murata"
+		(property "Manufacturer" "Taiyo Yuden"
 			(at 143.51 55.88 0)
 			(effects
@@
 			)
 		)
-		(property "MPN" "GRM21BR61E106KA73L"
+		(property "MPN" "TMK212BBJ106MG-T"
 			(at 293.37 88.9 0)
 			(effects
@@
 			)
 		)
-		(property "Manufacturer" "Murata"
+		(property "Manufacturer" "Taiyo Yuden"
 			(at 293.37 88.9 0)
 			(effects
@@
 			)
 		)
-		(property "MPN" "GRM21BR61E106KA73L"
+		(property "MPN" "TMK212BBJ106MG-T"
 			(at 184.15 106.68 0)
 			(effects
@@
 			)
 		)
-		(property "Manufacturer" "Murata"
+		(property "Manufacturer" "Taiyo Yuden"
 			(at 184.15 106.68 0)
 			(effects
