File: fmc.kicad_sch (KiCad schematic)
At the start: 35 parts, among them P1 ASP-134488-01, Q1 FDN335N, Q2 FDN335N, Q3 FDN335N

Commit message: Modified Power Filtering
- Removed FB1 & C136
- Added additional 1210 bypassing caps on main power inputs from FMC
- Changed SMPS output caps to the new 1210 22uF part
- Changed Input cap to LD0 U44 to the new 22uF part.
Parts:
- added C136, C147, C148: 22uF, Capacitor_SMD:C_1210_3225Metric, symbol Device:C_Small
Connections:
- net +12V_FMC: now also C136.1
- net GND: now also C136.2, C147.2, C148.2
- net VADJ: now also C148.1
- net VDD3P3V: now also C147.1

Commit message: Changes to Power Filtering
- Removed extra bulk caps on FMC power inputs
- Cleaned up some power routing between U22 & U44
- Made some vias larger for power tree connections
- Changed 22uF to a new 35V part
- Changed 10uF part to a new equivalent part due to OOS.
- Modified text near U27 on schematic for clarity
- Added notes on the power schematics showing effective capacitance of chosen bulk mlcc caps
Parts:
- removed C136, C147, C148: 22uF, Capacitor_SMD:C_1210_3225Metric, symbol Device:C_Small
- C34, C35, C79: footprint Capacitor_SMD:C_0805_2012Metric -> Capacitor_SMD:C_1210_3225Metric; MPN KGM21AR51E226MU -> GMK325BJ226MM-P; Manufacturer KYOCERA AVX -> Taiyo Yuden
