File: trigger-output-fmc.kicad_pcb (KiCad board)
At the start: 8 copper layers, 84 x 69 mm, 342 parts, among them J1 MMCX, J10 MMCX, J11 MMCX, J12 MMCX, J13 MMCX, J14 MMCX, J15 MMCX, J16 MMCX, J19 WP Jumper, J2 MMCX, J3 MMCX, J4 MMCX, J5 MMCX, J6 MMCX, J7 MMCX, J8 MMCX, J9 MMCX, P1 ASP-134488-01, Q1 FDN335N, Q2 FDN335N, Q3 FDN335N, T1 TCM2-43X+, T2 TCM2-43X+, T3 TCM2-43X+, T4 TCM2-43X+, U1 TLV3601, U10 SN74LVC2G126, U11 TLV3601, U12 SN74LVC2G126, U13 TLV3601, U14 SN74LVC2G126, U15 TLV3601, U16 SN74LVC2G126, U17 TLV3601, U18 SI5394, U19 SI5394, U2 TLV3601, U20 TLV75733PDBV, U21 TLV75718PDBV, U22 TPS563200, U23 74AVC4T245, U24 TLV75733PDBV, U25 74AVC4T245, U26 74LVC8T245, U27 74LVC8T245, U28 TLV75718PDBV, U29 SN74LVC2G126, U3 TLV3601, U30 TLV3601, U31 SN74LVC2G126, U32 TLV3601, U33 SN74LVC2G126, U34 TLV3601, U35 SN74LVC2G126, U36 TLV3601, U37 SN74LVC2G126, U38 TLV3601, U39 SN74LVC2G126, U4 SN74LVC2G126, U40 TLV3601, U41 SN74LVC2G126, U42 TLV3601, U43 SN74LVC2G126, U44 LP3855EMP-ADJ/NOPB, U48 SN74LVC2G126, U5 SN74LVC2G126, U6 TLV3601, U7 SN74LVC2G126, U8 TLV3601, U9 AT24C64D, Y1 CX3225SB48000D0FPJC1, Y2 CX3225SB48000D0FPJC1

Commit message: Changes to Power Filtering
- Removed extra bulk caps on FMC power inputs
- Cleaned up some power routing between U22 & U44
- Made some vias larger for power tree connections
- Changed 22uF to a new 35V part
- Changed 10uF part to a new equivalent part due to OOS.
- Modified text near U27 on schematic for clarity
- Added notes on the power schematics showing effective capacitance of chosen bulk mlcc caps
Parts:
- removed C136, C147, C148: 22uF, Capacitor_SMD:C_1210_3225Metric
- C34, C35, C79: footprint Capacitor_SMD:C_0805_2012Metric -> Capacitor_SMD:C_1210_3225Metric
- moved FB3 5.20 mm to (147.5, 132.7)
- moved C35 5.04 mm to (177.1, 133.5), turned to -90 degrees
- moved C54 3.72 mm to (151.9, 134.7), turned to -90 degrees
- moved C53 2.52 mm to (155.4, 134.7)
- moved R43 2.21 mm to (179.2, 137.0), turned to 180 degrees
- moved C79 1.40 mm to (174.0, 128.2), turned to 90 degrees
- moved C34 1.30 mm to (180.2, 125.9), turned to -90 degrees
- moved TP3 0.50 mm to (184.8, 129.0)
- moved C71 0.42 mm to (159.8, 132.3)
Routing:
- net /Digital IO/Switched_5P45V: track 99.0 -> 88.7 mm
- net +12V_FMC: track 25.5 -> 16.1 mm
- net Net-(U44-Vin): track 6.24 -> 14.1 mm, vias 1 -> 3
- net GND: track 535.3 -> 529.1 mm, vias 267 -> 261
- net Net-(H1-Pad1): track 4.85 -> 6.85 mm
- net VDD3P3V: track 49.2 -> 47.5 mm
- net /Digital IO/D_Output15.N: track 43.2 -> 41.9 mm
- net /Digital IO/D_Output15.P: track 42.3 -> 41.0 mm
- net VADJ: track 55.3 -> 55.8 mm
