File: trigger-output-fmc.kicad_pcb (KiCad board)
At the start: 8 copper layers, 84 x 69 mm, 339 parts, among them J1 MMCX, J10 MMCX, J11 MMCX, J12 MMCX, J13 MMCX, J14 MMCX, J15 MMCX, J16 MMCX, J19 WP Jumper, J2 MMCX, J3 MMCX, J4 MMCX, J5 MMCX, J6 MMCX, J7 MMCX, J8 MMCX, J9 MMCX, P1 ASP-134488-01, Q1 FDN335N, Q2 FDN335N, Q3 FDN335N, T1 TCM2-43X+, T2 TCM2-43X+, T3 TCM2-43X+, T4 TCM2-43X+, U1 TLV3601, U10 SN74LVC2G126, U11 TLV3601, U12 SN74LVC2G126, U13 TLV3601, U14 SN74LVC2G126, U15 TLV3601, U16 SN74LVC2G126, U17 TLV3601, U18 SI5394, U19 SI5394, U2 TLV3601, U20 TLV75733PDBV, U21 TLV75718PDBV, U22 TPS563200, U23 74AVC4T245, U24 TLV75733PDBV, U25 74AVC4T245, U26 74LVC8T245, U27 74LVC8T245, U28 TLV75718PDBV, U29 SN74LVC2G126, U3 TLV3601, U30 TLV3601, U31 SN74LVC2G126, U32 TLV3601, U33 SN74LVC2G126, U34 TLV3601, U35 SN74LVC2G126, U36 TLV3601, U37 SN74LVC2G126, U38 TLV3601, U39 SN74LVC2G126, U4 SN74LVC2G126, U40 TLV3601, U41 SN74LVC2G126, U42 TLV3601, U43 SN74LVC2G126, U44 LP3855EMP-ADJ/NOPB, U48 SN74LVC2G126, U5 SN74LVC2G126, U6 TLV3601, U7 SN74LVC2G126, U8 TLV3601, U9 AT24C64D, Y1 CX3225SB48000D0FPJC1, Y2 CX3225SB48000D0FPJC1

Commit message: Small tweaks to power filtering
-Removed C48
-Changed C49 to a 22uF 2010 part (up from 10uF)
- moved C79 (VADJ Bulk cap) to revert changes to LVDS Digital Output pairs.
- Added trace between 12VDC Decoupling cap and TP1
Parts:
- removed C48: 10uF, Capacitor_SMD:C_0805_2012Metric
- C49: value 10uF -> 22uF; footprint Capacitor_SMD:C_0805_2012Metric -> Capacitor_SMD:C_1210_3225Metric
- moved C35 4.00 mm to (180.3, 131.1)
- moved C79 2.90 mm to (174.0, 131.1)
- moved C49 1.00 mm to (164.7, 137.1)
Routing:
- net +12V_FMC: track 16.1 -> 21.5 mm
- net VADJ: track 55.8 -> 54.0 mm
- net /Digital IO/D_Output15.P: track 41.0 -> 42.3 mm
- net /Digital IO/D_Output15.N: track 41.9 -> 43.2 mm
- net VDD3P3V: track 47.5 -> 48.2 mm
- net GND: track 529.1 -> 529.0 mm, vias 261 -> 258
